Commit message: made the lidar move!

File: catkin_ws/src/mavs_description/urdf/lidar_example.urdf.xacro (robot description, xacro)
@@ -30,4 +30,4 @@
   <!-- Bolt-on sensors go here -->
   <xacro:include filename="$(find mavs_description)/urdf/lidar_vlp_16.urdf.xacro"/>
-  <xacro:lidar parent="base_link" name="velodyne" topic="/velodyne_points" x="0" y="0" z="0.4" roll="0" pitch="0" yaw="0" />
+  <xacro:lidar parent="base_link" name="velodyne" topic1="/speed" topic2="/velodyne_points" x="0" y="0" z="0.4" roll="0" pitch="0" yaw="0" />
 </robot>

File: catkin_ws/src/mavs_description/urdf/lidar_vlp_16.urdf.xacro (robot description, xacro)
@@ -2,5 +2,5 @@
 <robot xmlns:xacro="http://www.ros.org/wiki/xacro" name="VLP-16">
   <xacro:property name="M_PI" value="3.1415926535897931" />
-  <xacro:macro name="lidar" params="parent name topic x y z roll pitch yaw">
+  <xacro:macro name="lidar" params="parent name topic1 topic2 x y z roll pitch yaw">
     <joint name="${name}_base_mount_joint" type="fixed">
       <parent link="${parent}"/>
@@ -49,4 +49,10 @@
       </visual>
     </link>
+    <gazebo>
+      <!-- reference to plugin -->
+      <plugin name="model_push" filename="libmodel_push.so">
+          <topicName>${topic1}</topicName>
+      </plugin>
+    </gazebo>
     <!-- Gazebo requires the velodyne_gazebo_plugins package -->
     <gazebo reference="${name}">
@@ -82,5 +88,5 @@
         </ray>
         <plugin name="gazebo_ros_laser_controller" filename="libgazebo_ros_velodyne_laser.so">
-          <topicName>${topic}</topicName>
+          <topicName>${topic2}</topicName>
           <frameName>/${name}</frameName>
           <min_range>0.9</min_range>
