Commit message: added teliop example and move along x example

File: catkin_ws/src/mavs_description/urdf/velodyne_16.xacro (robot description, xacro)
@@ -1,12 +1,12 @@
 <?xml version="1.0"?>
-<robot xmlns:xacro="http://www.ros.org/wiki/xacro" name="VLP-16">
-  <xacro:property name="M_PI" value="3.1415926535897931" />
-  <xacro:macro name="lidar" params="parent name topic1 topic2 x y z roll pitch yaw">
-    <joint name="${name}_base_mount_joint" type="fixed">
+<robot name="velodyne_16" xmlns:xacro="http://www.ros.org/wiki/xacro" >
+  <xacro:macro name="velodyne_16" params="parent lidar_x lidar_z">
+    <joint name="velodyne_joint" type="fixed">
+      <axis xyz="${lidar_x} 0 ${lidar_z}" />
+      <origin xyz="${lidar_x} 0 ${lidar_z}" rpy="0 0 0" />
       <parent link="${parent}"/>
-      <child link="${name}_base_link"/>
-      <origin xyz="${x} ${y} ${z}" rpy="${roll} ${pitch} ${yaw}" />
+      <child link="velodyne_base_link"/>
     </joint>
-    <link name="${name}_base_link">
+    <link name="velodyne_base_link">
       <inertial>
         <mass value="0.1"/>
@@ -31,10 +31,10 @@
       </collision>
     </link>
-    <joint name="${name}_base_scan_joint" type="fixed" >
+    <joint name="scan_joint" type="fixed" >
       <origin xyz="0 0 0.0377" rpy="0 0 0" />
-      <parent link="${name}_base_link" />
-      <child link="${name}"/>
+      <parent link="velodyne_base_link" />
+      <child link="velodyne_top_link"/>
     </joint>
-    <link name="${name}">
+    <link name="velodyne_top_link">
       <inertial>
         <mass value="0.1"/>
@@ -49,15 +49,7 @@
       </visual>
     </link>
-    <gazebo>
-      <!-- reference to plugin -->
-      <!-- plugin name="model_push" filename="libmodel_push.so" -->
-      <plugin name="model_push" filename="libvelodyne_plugin.so">
-          <topicName>${topic1}</topicName>
-          <frameName>"push_frame"</frameName>
-      </plugin>
-    </gazebo>
     <!-- Gazebo requires the velodyne_gazebo_plugins package -->
-    <gazebo reference="${name}">
-      <sensor type="ray" name="${name}-VLP16">
+    <gazebo reference="velodyne_top_link">
+      <sensor type="ray" name="velodyne_16">
         <pose>0 0 0 0 0 0</pose>
         <visualize>false</visualize>
@@ -90,6 +82,6 @@
         </ray>
         <plugin name="gazebo_ros_laser_controller" filename="libgazebo_ros_velodyne_laser.so">
-          <topicName>${topic2}</topicName>
-          <frameName>/${name}</frameName>
+          <topicName>${topic}</topicName>
+          <frameName>/gazebo_laser</frameName>
           <min_range>0.9</min_range>
           <max_range>130.0</max_range>
