Commit message: started to add vehicle model

File: catkin_ws/src/mavs_description/urdf/block.xacro (robot description, xacro)
@@ -27,4 +27,45 @@
       </inertial>
     </link>
+    <link name="steer_fl">
+     <inertial>
+       <origin xyz="-0.013054 -0.0295 0" rpy="0 0 0"/>
+       <mass value="1.0"/>
+       <inertia ixx="0.037227" ixy="0" ixz="0" iyy="0.04" iyz="0" izz="0.06"/>
+     </inertial>
+   </link>
+    <link name="wheel_fl">
+      <inertial>
+        <origin xyz="0 0 0" rpy="0 -3.141593 0"/>
+        <mass value="10.0"/>
+        <inertia ixx="0.305583" ixy="0" ixz="0" iyy="0.305583" iyz="0" izz="0.5445"/>
+      </inertial>
+      <visual name="wheel_fl_visual">
+        <origin xyz="0 0 0.0385" rpy="-1.570796 -1.570796 0"/>
+        <geometry>
+          <mesh filename="package://mavs_description/meshes/wheel.dae" scale="0.01 0.01 0.01"/>
+        </geometry>
+        <material name="carpaint_002"/>
+      </visual>
+      <collision name="wheel_fl_collision">
+        <origin xyz="0 0 0" rpy="0 -3.141593 0"/>
+        <geometry>
+          <cylinder radius="0.33" length="0.2"/>
+        </geometry>
+      </collision>
+    </link>
+    <joint name="steer_fl" type="revolute">
+      <origin xyz="1.435054 0.817 0.33" rpy="0 0 0"/>
+      <parent link="${base_link}"/>
+      <child link="steer_fl"/>
+      <axis xyz="0 0 1.0"/>
+      <limit lower="-0.6" upper="0.6" effort="0" velocity="0"/>
+    </joint>
+    <joint name="wheel_fl" type="continuous">
+      <origin xyz="-0.012654 -0.0295 -0.33" rpy="1.570796 0 -3.141593"/>
+      <parent link="steer_fl"/>
+      <child link="wheel_fl"/>
+      <axis xyz="0 0 1.0"/>
+      <limit effort="0" velocity="22.0"/>
+    </joint>
     <!-- Link1 -->
     <gazebo reference="${base_link}">

File: catkin_ws/src/mavs_gazebo/urdf/mavs.urdf.xacro (robot description, xacro)
@@ -2,11 +2,8 @@
 <robot name="mavs" xmlns:xacro="http://www.ros.org/wiki/xacro" >
   <!-- Necessary includes -->
-  <!--
-  <xacro:include filename="$(find mavs_description)/urdf/vehicle_structure.urdf.xacro" />
+  <xacro:include filename="$(find mavs_description)/urdf/hwmmv.urdf.xacro" />
   <xacro:include filename="$(find mavs_description)/urdf/vehicle_gazebo.urdf.xacro" />
-  -->
   <!-- Bolt-on sensors go here -->
-  <xacro:include filename="$(find mavs_description)/urdf/sensors.urdf.xacro" />
-  <xacro:lidar name="lidar" parent_link="base_footprint" x="0.6" y="0" z="1.3" roll="0" pitch="0.6" yaw="0" />
-  <xacro:gps name="gps" parent_link="base_footprint" x="-0.8" y="0" z="1.45" rate="50.0" ref_lat="45.0" ref_lon="-81.0" />
+  <xacro:include filename="$(find mavs_description)/urdf/velodyne_16.xacro"/>
+  <velodyne_16 parent="${base_link}" lidar_x="${lidar_x}" lidar_z="${lidar_z}"/>
 </robot>
