Commit message: continue to work on vehilce model in Gazebo

File: catkin_ws/src/mavs_description/urdf/hmmwv.xacro (robot description, xacro)
@@ -1,183 +1,13 @@
 <?xml version="1.0"?>
-<!-- created with Phobos 0.7 -->
-  <robot name="dbw_mkz" xmlns:xacro="http://www.ros.org/wiki/xacro">
-    <xacro:arg name="dae_file" default="$(find mavs_description)/meshes/hwwmv.dae"/>
-    <link name="base_footprint">
-    </link>
-    <link name="base_link">
-      <inertial>
-        <origin xyz="0 0 0.25" rpy="0 0 0"/>
-        <mass value="1500.0"/>
-        <inertia ixx="1000.0" ixy="0" ixz="0" iyy="1000.0" iyz="0" izz="1000.0"/>
-      </inertial>
-      <visual name="chassis">
-        <origin xyz="-0.058415 0 -0.33" rpy="0 0 1.570796"/>
-        <geometry>
-          <mesh filename="file://$(arg dae_file)" scale="0.394 0.394 0.394"/>
-        </geometry>
-        <material name="black.001"/>
-      </visual>
-      <collision name="chassis_collision">
-        <origin xyz="0.084967 -0.03046 0.350609" rpy="1.570796 0 -3.141593"/>
-        <geometry>
-          <mesh filename="package://dbw_mkz_description/meshes/body_collision.stl" scale="0.001 0.001 0.001"/>
-        </geometry>
-      </collision>
-    </link>
-    <link name="steer_fl">
-      <inertial>
-        <origin xyz="-0.013054 -0.0295 0" rpy="0 0 0"/>
-        <mass value="1.0"/>
-        <inertia ixx="0.037227" ixy="0" ixz="0" iyy="0.04" iyz="0" izz="0.06"/>
-      </inertial>
-    </link>
-    <link name="steer_fr">
-      <inertial>
-        <origin xyz="-0.01305 0.0275 0" rpy="0 0 0"/>
-        <mass value="1.0"/>
-        <inertia ixx="0.037227" ixy="0" ixz="0" iyy="0.04" iyz="0" izz="0.06"/>
-      </inertial>
-    </link>
-    <link name="wheel_fl">
-      <inertial>
-        <origin xyz="0 0 0" rpy="0 -3.141593 0"/>
-        <mass value="10.0"/>
-        <inertia ixx="0.305583" ixy="0" ixz="0" iyy="0.305583" iyz="0" izz="0.5445"/>
-      </inertial>
-      <visual name="wheel_fl_visual">
-        <origin xyz="0 0 0.0385" rpy="-1.570796 -1.570796 0"/>
-        <geometry>
-          <mesh filename="package://mavs_description/meshes/wheel.dae"/>
-        </geometry>
-        <material name="carpaint_002"/>
-      </visual>
-      <collision name="wheel_fl_collision">
-        <origin xyz="0 0 0" rpy="0 -3.141593 0"/>
-        <geometry>
-          <cylinder radius="0.33" length="0.2"/>
-        </geometry>
-      </collision>
-    </link>
-    <link name="wheel_fr">
-      <inertial>
-        <origin xyz="0 0 0" rpy="0 3.141593 0"/>
-        <mass value="10.0"/>
-        <inertia ixx="0.305583" ixy="0" ixz="0" iyy="0.305583" iyz="0" izz="0.5445"/>
-      </inertial>
-      <visual name="wheel_fr_visual">
-        <origin xyz="0 0 -0.043777" rpy="-1.570796 1.570796 0"/>
-        <geometry>
-          <mesh filename="package://mavs_description/meshes/wheel.dae" />
-        </geometry>
-        <material name="carpaint_002.001"/>
-      </visual>
-      <collision name="wheel_fr_collision">
-        <origin xyz="0 0 -0.0035" rpy="0 3.141593 0"/>
-        <geometry>
-          <cylinder radius="0.33" length="0.2"/>
-        </geometry>
-      </collision>
-    </link>
-    <link name="wheel_rl">
-      <inertial>
-        <origin xyz="0 0 -0.021117" rpy="0 3.141593 0"/>
-        <mass value="10.0"/>
-        <inertia ixx="0.305583" ixy="0" ixz="0" iyy="0.305583" iyz="0" izz="0.5445"/>
-      </inertial>
-      <visual name="wheel_rl_visual">
-        <origin xyz="0 0 0.017382" rpy="-1.570796 -1.570796 0"/>
-        <geometry>
-          <mesh filename="package://mavs_description/meshes/wheel.dae" />
-        </geometry>
-        <material name="carpaint_002.003"/>
-      </visual>
-      <collision name="wheel_rl_collision">
-        <origin xyz="0 0 -0.021118" rpy="0 3.141593 0"/>
-        <geometry>
-          <cylinder radius="0.33" length="0.2"/>
-        </geometry>
-      </collision>
-    </link>
-    <link name="wheel_rr">
-      <inertial>
-        <origin xyz="0 0 0.0205" rpy="0 3.141593 0"/>
-        <mass value="10.0"/>
-        <inertia ixx="0.305583" ixy="0" ixz="0" iyy="0.305583" iyz="0" izz="0.5445"/>
-      </inertial>
-      <visual name="wheel_rr_visual">
-        <origin xyz="0 0 -0.019214" rpy="-1.570796 1.570796 0"/>
-        <geometry>
-          <mesh filename="package://mavs_description/meshes/wheel.dae" scale="0.01 0.01 0.01"/>
-        </geometry>
-        <material name="carpaint_002.002"/>
-      </visual>
-      <collision name="wheel_rr_collision">
-        <origin xyz="0 0 0.0205" rpy="0 3.141593 0"/>
-        <geometry>
-          <cylinder radius="0.33" length="0.2"/>
-        </geometry>
-      </collision>
-    </link>
-    <joint name="base_link" type="fixed">
-      <origin xyz="0 0 0.33" rpy="0 0 0"/>
-      <parent link="base_footprint"/>
-      <child link="base_link"/>
-    </joint>
-    <joint name="steer_fl" type="revolute">
-      <origin xyz="1.435054 0.817 0.33" rpy="0 0 0"/>
-      <parent link="base_link"/>
-      <child link="steer_fl"/>
-      <axis xyz="0 0 1.0"/>
-      <limit lower="-0.6" upper="0.6" effort="0" velocity="0"/>
-    </joint>
-    <joint name="steer_fr" type="revolute">
-      <origin xyz="1.43505 -0.815 0.33" rpy="0 0 0"/>
-      <parent link="base_link"/>
-      <child link="steer_fr"/>
-      <axis xyz="0 0 1.0"/>
-      <limit lower="-0.6" upper="0.6" effort="0" velocity="0"/>
-    </joint>
-    <joint name="wheel_fl" type="continuous">
-      <origin xyz="-0.012654 -0.0295 -0.33" rpy="1.570796 0 -3.141593"/>
-      <parent link="steer_fl"/>
-      <child link="wheel_fl"/>
-      <axis xyz="0 0 1.0"/>
-      <limit effort="0" velocity="22.0"/>
-    </joint>
-    <joint name="wheel_fr" type="continuous">
-      <origin xyz="-0.01265 0.0275 -0.33" rpy="1.570796 0 -3.141593"/>
-      <parent link="steer_fr"/>
-      <child link="wheel_fr"/>
-      <axis xyz="0 0 1.0"/>
-      <limit effort="0" velocity="22.0"/>
-    </joint>
-    <joint name="wheel_rl" type="continuous">
-      <origin xyz="-1.4224 0.808618 0" rpy="1.570796 0 -3.141593"/>
-      <parent link="base_link"/>
-      <child link="wheel_rl"/>
-      <axis xyz="0 0 1.0"/>
-      <limit effort="5000.0" velocity="22.0"/>
-    </joint>
-    <joint name="wheel_rr" type="continuous">
-      <origin xyz="-1.4224 -0.808 0" rpy="1.570796 0 -3.141593"/>
-      <parent link="base_link"/>
-      <child link="wheel_rr"/>
-      <axis xyz="0 0 1.0"/>
-      <limit effort="5000.0" velocity="22.0"/>
-    </joint>
-    <material name="black.001">
-      <color rgba="0 0 0 1.0"/>
-    </material>
-    <material name="carpaint_002">
-      <color rgba="0.941177 0.941177 0.941177 1.0"/>
-    </material>
-    <material name="carpaint_002.001">
-      <color rgba="0.941177 0.941177 0.941177 1.0"/>
-    </material>
-    <material name="carpaint_002.002">
-      <color rgba="0.941177 0.941177 0.941177 1.0"/>
-    </material>
-    <material name="carpaint_002.003">
-      <color rgba="0.941177 0.941177 0.941177 1.0"/>
-    </material>
-  </robot>
+<robot name="front_wheel" xmlns:xacro="http://www.ros.org/wiki/xacro" >
+  <!-- Vehicle modeled as a giant block -->
+  <xacro:include filename="$(find mavs_description)/urdf/body.xacro"/>
+  <block base_link="${base_link}">
+    <xacro:insert_block name="base_geometry" />
+  </block>
+  <xacro:include filename="$(find mavs_description)/urdf/wheel.xacro"/>
+  <xacro:wheel fb="front" lr="right" parent="base_link"/>
+  <xacro:wheel fb="front" lr="left" parent="base_link"/>
+  <xacro:wheel fb="rear" lr="right" parent="base_link"/>
+  <xacro:wheel fb="rear" lr="left" parent="base_link"/>
+</robot>
