Commit message: added tf from world to base_link

File: catkin_ws/src/mavs_description/urdf/body.xacro (robot description, xacro)
@@ -1,22 +1,8 @@
 <?xml version="1.0"?>
 <robot xmlns:xacro="http://www.ros.org/wiki/xacro">
-  <xacro:macro name="block" params="base_link *base_geometry">
+  <xacro:macro name="body" params="base_link *base_geometry">
     <!-- Base Footprint -->
     <!-- base_footprint is a fictitious link(frame) that is on the ground right below base_link origin -->
-    <link name="base_footprint">
-      <inertial>
-        <mass value="0.0001" />
-        <origin xyz="0 0 0" />
-        <inertia ixx="0.0001" ixy="0.0" ixz="0.0"
-            iyy="0.0001" iyz="0.0"
-            izz="0.0001" />
-      </inertial>
-      <visual>
-        <origin xyz="0 0 0" rpy="0 0 0" />
-        <geometry>
-            <box size="0.001 0.001 0.001" />
-        </geometry>
-      </visual>
-    </link>
+    <link name="base_footprint"/>
    <gazebo reference="base_footprint">
      <turnGravityOff>false</turnGravityOff>

File: catkin_ws/src/mavs_description/urdf/hmmwv.xacro (robot description, xacro)
@@ -1,9 +1,9 @@
 <?xml version="1.0"?>
-<robot name="front_wheel" xmlns:xacro="http://www.ros.org/wiki/xacro" >
+<robot name="hmmwv" xmlns:xacro="http://www.ros.org/wiki/xacro" >
   <!-- Vehicle modeled as a giant block -->
   <xacro:include filename="$(find mavs_description)/urdf/body.xacro"/>
-  <block base_link="${base_link}">
+  <body base_link="${base_link}">
     <xacro:insert_block name="base_geometry" />
-  </block>
+  </body>
   <xacro:include filename="$(find mavs_description)/urdf/wheel.xacro"/>
   <xacro:wheel fb="front" lr="right" parent="base_link"/>

File: catkin_ws/src/mavs_description/urdf/vehicle_gazebo.urdf.xacro (robot description, xacro)
@@ -22,3 +22,10 @@
     <mu2>${wheel_friction}</mu2>
   </gazebo>
+  <!-- ros_control plugin -->
+  <gazebo>
+    <plugin name="gazebo_ros_control" filename="libgazebo_ros_control.so">
+      <robotNamespace>/mavs</robotNamespace>
+      <robotSimType>gazebo_ros_control/DefaultRobotHWSim</robotSimType>
+    </plugin>
+  </gazebo>
 </robot>

File: catkin_ws/src/mavs_description/urdf/wheel.xacro (robot description, xacro)
@@ -86,7 +86,9 @@
       <transmission name="steer_${lr}_wheel_joint_trans">
         <type>transmission_interface/SimpleTransmission</type>
-        <joint name="steer_${lr}_wheel_joint" />
+        <joint name="steer_${lr}_wheel_joint">
+          <hardwareInterface>hardware_interface/EffortJointInterface</hardwareInterface>
+        </joint>
         <actuator name="${lr}_wheel_joint_motor">
-          <hardwareInterface>EffortJointInterface</hardwareInterface>
+          <hardwareInterface>hardware_interface/EffortJointInterface</hardwareInterface>
           <mechanicalReduction>1</mechanicalReduction>
         </actuator>
@@ -96,7 +98,9 @@
     <transmission name="${fb}_${lr}_wheel_joint_trans">
       <type>transmission_interface/SimpleTransmission</type>
-      <joint name="${fb}_${lr}_wheel_joint" />
+      <joint name="${fb}_${lr}_wheel_joint">
+        <hardwareInterface>hardware_interface/EffortJointInterface</hardwareInterface>
+      </joint>
       <actuator name="${fb}_${lr}_wheel_joint_motor">
-        <hardwareInterface>EffortJointInterface</hardwareInterface>
+        <hardwareInterface>hardware_interface/EffortJointInterface</hardwareInterface>
         <mechanicalReduction>1</mechanicalReduction>
       </actuator>

Commit message: started to implement yaml files, for obstacles and initial vehicle state

File: catkin_ws/src/mavs_description/urdf/body.xacro (robot description, xacro)
@@ -9,5 +9,5 @@
    </gazebo>
     <joint name="joint1" type="fixed" >
-      <origin xyz="0 0 ${base_clearance}" rpy="0 0 0" />
+      <origin xyz="${x0} ${y0} ${base_clearance}" rpy="0 0 ${psi0}" />
       <parent link="base_footprint" />
       <child link="${base_link}" />
@@ -18,5 +18,5 @@
       <visual>
         <xacro:if value="${mesh_mode == 1}">
-          <origin xyz="0 0 ${-wheel_radius}" rpy="0 0 ${M_PI}" />
+          <origin xyz="0 0 ${-wheel_radius}" rpy="0 0 ${pi}" />
           <geometry>
             <mesh filename="package://mavs_description/meshes/body.dae" scale=" ${scale_factor} ${scale_factor} ${scale_factor}"/>

File: catkin_ws/src/mavs_description/urdf/hmmwv.xacro (robot description, xacro)
@@ -1,5 +1,5 @@
 <?xml version="1.0"?>
 <robot name="hmmwv" xmlns:xacro="http://www.ros.org/wiki/xacro" >
-  <!-- Vehicle modeled as a giant block -->
+  <!-- Vehicle body-->
   <xacro:include filename="$(find mavs_description)/urdf/body.xacro"/>
   <body base_link="${base_link}">

File: catkin_ws/src/mavs_description/urdf/velodyne_16.xacro (robot description, xacro)
@@ -60,12 +60,12 @@
               <samples>1875</samples>
               <resolution>1</resolution>
-              <min_angle>-${M_PI}</min_angle>
-              <max_angle> ${M_PI}</max_angle>
+              <min_angle>-${pi}</min_angle>
+              <max_angle> ${pi}</max_angle>
             </horizontal>
             <vertical>
               <samples>16</samples>
               <resolution>1</resolution>
-              <min_angle>-${15.0*M_PI/180.0}</min_angle>
-              <max_angle> ${15.0*M_PI/180.0}</max_angle>
+              <min_angle>-${15.0*pi/180.0}</min_angle>
+              <max_angle> ${15.0*pi/180.0}</max_angle>
             </vertical>
           </scan>

File: catkin_ws/src/mavs_description/urdf/wheel.xacro (robot description, xacro)
@@ -16,5 +16,5 @@
         </xacro:if>
         <xacro:if value="${mesh_mode == 0}">
-          <origin xyz="0 0 0" rpy="${M_PI/2} 0 0" />
+          <origin xyz="0 0 0" rpy="${pi/2} 0 0" />
           <geometry>
             <cylinder length="${wheel_width}" radius="${wheel_radius}" />
@@ -24,5 +24,5 @@
       </visual>
       <collision>
-        <origin xyz="0 0 0" rpy="${M_PI/2} 0 0 " />
+        <origin xyz="0 0 0" rpy="${pi/2} 0 0 " />
         <geometry>
           <cylinder length="${wheel_width}" radius="${wheel_radius}" />
@@ -31,5 +31,5 @@
       <inertial>
         <mass value="${wheel_mass}" />
-        <origin xyz="0 0 0 "  rpy="${M_PI/2} 0 0" />
+        <origin xyz="0 0 0 "  rpy="${pi/2} 0 0" />
         <xacro:cylinder_inertia  m="${wheel_mass}" r="${wheel_radius}" h="${wheel_width}" />
       </inertial>
@@ -52,5 +52,5 @@
         <parent link="${parent}"/>
         <xacro:if value="${lr == 'right'}">
-          <origin xyz="${-lb} ${-wheel_base} 0" rpy="0 0 ${M_PI}" />
+          <origin xyz="${-lb} ${-wheel_base} 0" rpy="0 0 ${pi}" />
         </xacro:if>
         <xacro:if value="${lr == 'left'}">
@@ -73,5 +73,5 @@
       <joint name="steer_${lr}_wheel_joint" type="revolute">
         <xacro:if value="${lr == 'right'}">
-          <origin xyz="${la} ${-wheel_base} 0" rpy="0 0 ${M_PI}" />
+          <origin xyz="${la} ${-wheel_base} 0" rpy="0 0 ${pi}" />
         </xacro:if>
         <xacro:if value="${lr == 'left'}">

Commit message: made files more parametric

File: catkin_ws/src/mavs_description/urdf/body.xacro (robot description, xacro)
@@ -5,7 +5,4 @@
     <!-- base_footprint is a fictitious link(frame) that is on the ground right below base_link origin -->
     <link name="base_footprint"/>
-   <gazebo reference="base_footprint">
-     <turnGravityOff>false</turnGravityOff>
-   </gazebo>
     <joint name="joint1" type="fixed" >
       <origin xyz="${x0} ${y0} ${base_clearance}" rpy="0 0 ${psi0}" />
@@ -29,13 +26,12 @@
       </visual>
       <collision>
+        <!--selfCollide>false</selfCollide-->
         <origin xyz="0 0 ${base_height/2}" rpy="0 0 0" />
         <xacro:insert_block name="base_geometry" />
       </collision>
       <inertial>
-        <mass value="10"/>
+        <mass value="1500"/>
         <origin xyz="0 0 ${base_height/2}" rpy="0 0 0"/>
-        <inertia ixx="3.0" ixy="0.0" ixz="0.0"
-                 iyy="3.0" iyz="0.0"
-                 izz="3.0" />
+        <inertia ixx="1000.0" ixy="0" ixz="0" iyy="1000.0" iyz="0" izz="1000.0"/>
       </inertial>
     </link>

File: catkin_ws/src/mavs_description/urdf/obstacles.urdf.xacro (robot description, xacro)
@@ -3,12 +3,11 @@
   <!-- obstacles-->
   <xacro:include filename="$(find mavs_description)/urdf/obstacle.urdf.xacro"/>
-  <xacro:property name="sim_params_file" value="$(find mavs_gazebo)/config/default_sim_params.yaml"/>
-  <xacro:property name="sim" value="${load_yaml(sim_params_file)}"/>
-  <xacro:property name="radius" value="${sim['mavs']['obs']['radius']}" />
-  <xacro:property name="length" value="${sim['mavs']['obs']['length']}" />
-  <xacro:property name="x0" value="${sim['mavs']['obs']['x0']}" />
-  <xacro:property name="y0" value="${sim['mavs']['obs']['y0']}" />
+  <xacro:property name="mavs_params_file" value="$(find mavs_gazebo)/config/mavs_params.yaml"/>
+  <xacro:property name="mavs" value="${load_yaml(mavs_params_file)}"/>
+  <xacro:property name="radius" value="${mavs['mavs']['obs']['radius']}" />
+  <xacro:property name="length" value="${mavs['mavs']['obs']['length']}" />
+  <xacro:property name="x0" value="${mavs['mavs']['obs']['x0']}" />
+  <xacro:property name="y0" value="${mavs['mavs']['obs']['y0']}" />
   <obstacle idx="0"/>
-  <!-- xacro:obstacle/-->
 </robot>
 <!--TODO add speed-->

File: catkin_ws/src/mavs_description/urdf/vehicle_gazebo.urdf.xacro (robot description, xacro)
@@ -1,31 +1,44 @@
 <?xml version="1.0"?>
 <robot name="mavs_gazebo" xmlns:xacro="http://www.ros.org/wiki/xacro">
-  <xacro:property name="wheel_friction" value="1.2" />
-  <gazebo reference="base_link" >
-    <mu1>0.5</mu1>
-    <mu2>0.5</mu2>
-  </gazebo>
+  <!--- Surface properties -->
   <gazebo reference="wheel_fl" >
-    <mu1>${wheel_friction}</mu1>
-    <mu2>${wheel_friction}</mu2>
+    <mu1>${mu1}</mu1>
+    <mu2>${mu2}</mu2>
+    <minDepth>${minDepth}</minDepth>
+    <kp>${kp}</kp>
   </gazebo>
   <gazebo reference="wheel_fr" >
-    <mu1>${wheel_friction}</mu1>
-    <mu2>${wheel_friction}</mu2>
+    <mu1>${mu1}</mu1>
+    <mu2>${mu2}</mu2>
+    <minDepth>${minDepth}</minDepth>
+    <kp>${kp}</kp>
   </gazebo>
   <gazebo reference="wheel_rl" >
-    <mu1>${wheel_friction}</mu1>
-    <mu2>${wheel_friction}</mu2>
+    <mu1>${mu1}</mu1>
+    <mu2>${mu2}</mu2>
+    <minDepth>${minDepth}</minDepth>
+    <kp>${kp}</kp>
   </gazebo>
   <gazebo reference="wheel_rr" >
-    <mu1>${wheel_friction}</mu1>
-    <mu2>${wheel_friction}</mu2>
+    <mu1>${mu1}</mu1>
+    <mu2>${mu2}</mu2>
+    <minDepth>${minDepth}</minDepth>
+    <kp>${kp}</kp>
   </gazebo>
   <!-- ros_control plugin -->
   <gazebo>
     <plugin name="gazebo_ros_control" filename="libgazebo_ros_control.so">
-      <robotNamespace>/mavs</robotNamespace>
+      <robotNamespace>${robotNamespace}</robotNamespace>
       <robotSimType>gazebo_ros_control/DefaultRobotHWSim</robotSimType>
     </plugin>
   </gazebo>
+  <gazebo>
+    <plugin name="p3d" filename="libgazebo_ros_p3d.so">
+      <!-- <robotNamespace>/hmmwv</robotNamespace> -->
+      <bodyName>${base_link}</bodyName>
+      <topicName>${ground_truth_topic}</topicName>
+      <frameName>${map}</frameName>
+      <updateRate>100.0</updateRate>
+    </plugin>
+ </gazebo>
 </robot>

File: catkin_ws/src/mavs_description/urdf/wheel.xacro (robot description, xacro)
@@ -28,4 +28,5 @@
           <cylinder length="${wheel_width}" radius="${wheel_radius}" />
         </geometry>
+        <!--selfCollide>false</selfCollide-->
       </collision>
       <inertial>

File: catkin_ws/src/mavs_gazebo/urdf/mavs.urdf.xacro (robot description, xacro)
@@ -1,12 +1,19 @@
 <?xml version="1.0"?>
 <robot name="mavs" xmlns:xacro="http://www.ros.org/wiki/xacro" >
-  <xacro:property name="hmmwv_params_file" value="$(find mavs_description)/config/hmmwv_params.yaml"/>
-  <xacro:property name="vehicle" value="${load_yaml(hmmwv_params_file)}"/>
-  <xacro:property name="sim_params_file" value="$(find mavs_gazebo)/config/default_sim_params.yaml"/>
-  <xacro:property name="sim" value="${load_yaml(sim_params_file)}"/>
+  <xacro:property name="global_params_file" value="$(find mavs_gazebo)/config/global_params.yaml"/>
+  <xacro:property name="global_params" value="${load_yaml(global_params_file)}"/>
+  <xacro:property name="vehicle_params_file" value="$(find mavs_description)/config/hmmwv_params.yaml"/>
+  <xacro:property name="vehicle" value="${load_yaml(vehicle_params_file)}"/>
+  <xacro:property name="mavs_params_file" value="$(find mavs_gazebo)/config/mavs_params.yaml"/>
+  <xacro:property name="mavs" value="${load_yaml(mavs_params_file)}"/>
+  <!-- Frames, topics and names -->
+  <xacro:property name="robotNamespace" value="${global_params['robotNamespace']}" />
+  <xacro:property name="robotName" value="${global_params['robotName']}" />
+  <xacro:property name="map" value="${global_params['map']}" />
+  <xacro:property name="ground_truth_topic" value="${global_params['ground_truth_topic']}" />
   <!-- initial vehicle states -->
-  <xacro:property name="x0" value="${sim['mavs']['X0']['x']}" />
-  <xacro:property name="y0" value="${sim['mavs']['X0']['y']}" />
-  <xacro:property name="psi0" value="${sim['mavs']['X0']['psi']}" />
+  <xacro:property name="x0" value="${mavs['mavs']['X0']['x']}" />
+  <xacro:property name="y0" value="${mavs['mavs']['X0']['y']}" />
+  <xacro:property name="psi0" value="${mavs['mavs']['X0']['psi']}" />
   <xacro:property name="scale_factor" value="${vehicle['scale_factor']}" />
   <xacro:property name="mesh_mode" value="1"/>
@@ -29,4 +36,8 @@
   <xacro:property name="lb" value="${vehicle['lb']}"/>
   <xacro:property name="wheel_base" value="${vehicle['wheel_base']}" />
+  <xacro:property name="mu1" value="${vehicle['mu1']}" />
+  <xacro:property name="mu2" value="${vehicle['mu2']}" />
+  <xacro:property name="minDepth" value="${vehicle['minDepth']}" />
+  <xacro:property name="kp" value="${vehicle['kp']}" />
   <!-- LiDAR properties -->
   <xacro:property name="lidar_z" value="${vehicle['lidar_z']}"/>
