Commit message: updated so that vehicle can start at zero speed
added functionality to get obstacle data from Gazebo

File: catkin_ws/src/mavs_gazebo/urdf/mavs.xacro (robot description, xacro)
@@ -23,6 +23,6 @@
   <xacro:property name="wheel_base" value="1" />
   <!-- LiDAR properties -->
-  <xacro:property name="lidar_z" value="${base_height/2 + 0.1}" />
-  <xacro:property name="lidar_x" value="${base_length/2-0.1}" />
+  <xacro:property name="lidar_z" value="${base_height/2 + 0.5}" />
+  <xacro:property name="lidar_x" value="${base_length/2 + 0.1}" />
   <xacro:property name="topic" value="/lidar_points" />
   <!-- Necessary includes -->
